File: src/SMD-Heart.kicad_pcb (KiCad board)
At the start: 2 copper layers, 30.7 x 27.3 mm, 53 parts, among them Q1 FDG1024NZ, Q2 FDG1024NZ, Q3 FDG1024NZ, Q4 FDG1024NZ, Q5 FDG1024NZ, Q6 FDG1024NZ, Q7 FDG1024NZ

Commit message: modified 3D stuff
Routing:
- net GND: track 33.7 -> 32.1 mm
Other:
- board text added: "MY HEART BLINKS FOR YOU"
- board text removed: "Sample Text"
Changed lines of the file:
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@@
       (outputformat 1)
       (mirror false)
-      (drillshape 1)
+      (drillshape 0)
       (scaleselection 1)
-      (outputdirectory ""))
+      (outputdirectory ../grb/))
   )
   (net 0 "")
@@
     (pad 2 smd rect (at 0.874999 0 315) (size 0.67 1) (layers F.Cu F.Paste F.Mask)
       (net 28 "Net-(D7-Pad2)"))
-    (model ${KIPRJMOD}/3D/LED_0603.wrl
+    (model ${KISYS3DMOD}/LED_SMD.3dshapes/LED_0603_1608Metric.wrl
       (at (xyz 0 0 0))
       (scale (xyz 1 1 1))
@@
     (pad 2 smd rect (at 0.874999 0 45) (size 0.67 1) (layers F.Cu F.Paste F.Mask)
       (net 21 "Net-(D4-Pad2)"))
-    (model ${KIPRJMOD}/3D/LED_0603.wrl
+    (model ${KISYS3DMOD}/LED_SMD.3dshapes/LED_0603_1608Metric.wrl
       (at (xyz 0 0 0))
       (scale (xyz 1 1 1))
@@
     (pad 1 smd rect (at -0.874999 0 45) (size 0.67 1) (layers F.Cu F.Paste F.Mask)
       (net 35 "Net-(D11-Pad1)"))
-    (model ${KIPRJMOD}/3D/LED_0603.wrl
+    (model ${KISYS3DMOD}/LED_SMD.3dshapes/LED_0603_1608Metric.wrl
       (at (xyz 0 0 0))
       (scale (xyz 1 1 1))
@@
     (pad 2 smd rect (at 0.875 0 180) (size 0.67 1) (layers F.Cu F.Paste F.Mask)
       (net 44 "Net-(D13-Pad2)"))
-    (model ${KIPRJMOD}/3D/LED_0603.wrl
+    (model ${KISYS3DMOD}/LED_SMD.3dshapes/LED_0603_1608Metric.wrl
       (at (xyz 0 0 0))
       (scale (xyz 1 1 1))
@@
     (pad 1 smd rect (at -0.875 0 180) (size 0.67 1) (layers F.Cu F.Paste F.Mask)
       (net 16 "Net-(D1-Pad1)"))
-    (model ${KIPRJMOD}/3D/LED_0603.wrl
+    (model ${KISYS3DMOD}/LED_SMD.3dshapes/LED_0603_1608Metric.wrl
       (at (xyz 0 0 0))
       (scale (xyz 1 1 1))
@@
     (pad 2 smd rect (at 0.874999 0 135) (size 0.67 1) (layers F.Cu F.Paste F.Mask)
       (net 18 "Net-(D2-Pad2)"))
-    (model ${KIPRJMOD}/3D/LED_0603.wrl
+    (model ${KISYS3DMOD}/LED_SMD.3dshapes/LED_0603_1608Metric.wrl
       (at (xyz 0 0 0))
       (scale (xyz 1 1 1))
@@
     (pad 1 smd rect (at -0.875 0 90) (size 0.67 1) (layers F.Cu F.Paste F.Mask)
       (net 20 "Net-(D3-Pad1)"))
-    (model ${KIPRJMOD}/3D/LED_0603.wrl
+    (model ${KISYS3DMOD}/LED_SMD.3dshapes/LED_0603_1608Metric.wrl
       (at (xyz 0 0 0))
       (scale (xyz 1 1 1))
@@
     (pad 2 smd rect (at 0.874999 0 225) (size 0.67 1) (layers F.Cu F.Paste F.Mask)
       (net 24 "Net-(D5-Pad2)"))
-    (model ${KIPRJMOD}/3D/LED_0603.wrl
+    (model ${KISYS3DMOD}/LED_SMD.3dshapes/LED_0603_1608Metric.wrl
       (at (xyz 0 0 0))
       (scale (xyz 1 1 1))
@@
     (pad 1 smd rect (at -0.874999 0 225) (size 0.67 1) (layers F.Cu F.Paste F.Mask)
       (net 26 "Net-(D6-Pad1)"))
-    (model ${KIPRJMOD}/3D/LED_0603.wrl
+    (model ${KISYS3DMOD}/LED_SMD.3dshapes/LED_0603_1608Metric.wrl
       (at (xyz 0 0 0))
       (scale (xyz 1 1 1))
@@
     (pad 1 smd rect (at -0.874999 0 315) (size 0.67 1) (layers F.Cu F.Paste F.Mask)
       (net 30 "Net-(D8-Pad1)"))
-    (model ${KIPRJMOD}/3D/LED_0603.wrl
+    (model ${KISYS3DMOD}/LED_SMD.3dshapes/LED_0603_1608Metric.wrl
       (at (xyz 0 0 0))
       (scale (xyz 1 1 1))
@@
     (pad 2 smd rect (at 0.874999 0 135) (size 0.67 1) (layers F.Cu F.Paste F.Mask)
       (net 32 "Net-(D9-Pad2)"))
-    (model ${KIPRJMOD}/3D/LED_0603.wrl
+    (model ${KISYS3DMOD}/LED_SMD.3dshapes/LED_0603_1608Metric.wrl
       (at (xyz 0 0 0))
       (scale (xyz 1 1 1))
@@
     (pad 1 smd rect (at -0.875 0 90) (size 0.67 1) (layers F.Cu F.Paste F.Mask)
       (net 34 "Net-(D10-Pad1)"))
-    (model ${KIPRJMOD}/3D/LED_0603.wrl
+    (model ${KISYS3DMOD}/LED_SMD.3dshapes/LED_0603_1608Metric.wrl
       (at (xyz 0 0 0))
       (scale (xyz 1 1 1))
@@
     (pad 2 smd rect (at 0.875 0) (size 0.67 1) (layers F.Cu F.Paste F.Mask)
       (net 37 "Net-(D12-Pad2)"))
-    (model ${KIPRJMOD}/3D/LED_0603.wrl
+    (model ${KISYS3DMOD}/LED_SMD.3dshapes/LED_0603_1608Metric.wrl
       (at (xyz 0 0 0))
       (scale (xyz 1 1 1))
@@
     (pad 1 np_thru_hole circle (at 0 0) (size 1 1) (drill 0.5) (layers *.Cu *.Mask))
   )
-  (gr_text "Sample\nText" (at 76.2 42.545) (layer F.SilkS)
-    (effects (font (size 1.5 1.5) (thickness 0.3)))
+  (gr_text "MY HEART\nBLINKS\nFOR\nYOU" (at 76.2 44.069) (layer F.SilkS)
+    (effects (font (size 1.6 1.5) (thickness 0.3)))
   )
   (gr_arc (start 76.2 54.61) (end 74.93 55.88) (angle -90) (layer Edge.Cuts) (width 0.15))
@@
   (gr_line (start 77.47 55.88) (end 88.9 44.45) (layer Edge.Cuts) (width 0.15))
   (gr_line (start 74.93 55.88) (end 63.5 44.45) (layer Edge.Cuts) (width 0.15))
-  (segment (start 76.2 40.64) (end 76.2 48.133) (width 0.25) (layer B.Cu) (net 1))
-  (via (at 76.2 48.133) (size 0.8) (drill 0.4) (layers F.Cu B.Cu) (net 1))
+  (segment (start 76.2 40.64) (end 76.2 46.608996) (width 0.25) (layer B.Cu) (net 1))
+  (via (at 76.2 46.608996) (size 0.8) (drill 0.4) (layers F.Cu B.Cu) (net 1))
   (segment (start 68.9 35.164) (end 68.27518 35.164) (width 0.25) (layer F.Cu) (net 1))
   (segment (start 68.27518 35.164) (end 67.10159 33.99041) (width 0.25) (layer F.Cu) (net 1))
